File: AC-DC Switching/AC-DC Switching.kicad_pcb (KiCad board)
At the start: 2 copper layers, 24 parts, among them J3 12VDC, J4 0VDC, J5 DC_OUT, U1 TNY267P, U2 PC817

Commit message: update folders and files
Parts:
- removed J3: 12VDC, TestPoint:TestPoint_Pad_D1.0mm
- added Hm1: MountingHole, MountingHole:MountingHole_3.2mm_M3, F.Cu at (56.1, 58.3)
- added Hm2: MountingHole, MountingHole:MountingHole_3.2mm_M3, F.Cu at (156.2, 98.4)
- added Hm3: MountingHole, MountingHole:MountingHole_3.2mm_M3, F.Cu at (56.1, 98.3)
- added Hm4: MountingHole, MountingHole:MountingHole_3.2mm_M3, F.Cu at (156.2, 58.4)
- added J2: DC_OUT, Connector_Molex:Molex_KK-254_AE-6410-02A_1x02_P2.54mm_Vertical, F.Cu at (156.0, 67.2)
- added L1: 10u@3A, Inductor_THT:L_Toroid_Vertical_L21.6mm_W9.1mm_P8.40mm_Bourns_5700, F.Cu at (149.4, 83.2)
- added T1: EE22, Transformer_THT:Transformer_Myrra_EF20_7408x, F.Cu at (105.5, 64.9)
- C1: value 100uF/35V -> 2.2u@1kV; footprint Capacitor_THT:CP_Radial_D10.0mm_P5.00mm -> Capacitor_THT:C_Disc_D10.5mm_W5.0mm_P5.00mm
- C2: value 47uF/400V -> 47u@400V
- C3: value 0.1uF/50V -> 1000u@10V; footprint Capacitor_THT:C_Rect_L7.2mm_W3.5mm_P5.00mm_FKS2_FKP2_MKS2_MKP2 -> Capacitor_THT:CP_Radial_D12.5mm_P5.00mm
- C4: value 2.2uF/1kV -> 1000u@10V; footprint Capacitor_THT:C_Disc_D10.5mm_W5.0mm_P5.00mm -> Capacitor_THT:CP_Radial_D12.5mm_P5.00mm
- C5: value 1000uF/10V -> 100u@35V; footprint Capacitor_THT:CP_Radial_D12.5mm_P5.00mm -> Capacitor_THT:CP_Radial_D10.0mm_P5.00mm
- C6: value 1000uF/10V -> 0.1uF/50V; footprint Capacitor_THT:CP_Radial_D12.5mm_P5.00mm -> Capacitor_THT:C_Rect_L7.2mm_W3.5mm_P5.00mm_FKS2_FKP2_MKS2_MKP2
- D1: value LED -> DF04M; footprint LED_THT:LED_D3.0mm -> Diode_THT:Diode_Bridge_DIP-4_W7.62mm_P5.08mm
- D2: value DF04M -> LED; footprint Diode_THT:Diode_Bridge_DIP-4_W7.62mm_P5.08mm -> LED_THT:LED_D3.0mm
- D3: value 1N4148 -> 1N5822; footprint Diode_THT:D_DO-34_SOD68_P7.62mm_Horizontal -> Diode_THT:D_DO-201AD_P15.24mm_Horizontal
- D5: value 1N5822 -> 1N4148; footprint Diode_THT:D_DO-201AD_P15.24mm_Horizontal -> Diode_THT:D_DO-34_SOD68_P7.62mm_Horizontal
- J4: value 0VDC -> 12VDC
- J5: value DC_OUT -> 0VDC; footprint Connector_Molex:Molex_KK-254_AE-6410-02A_1x02_P2.54mm_Vertical -> TestPoint:TestPoint_Pad_D1.0mm
- R2: value 10k -> 200k
- R5: value 200k -> 59R
- R6: value 59 -> 10k
- R7: value 680 -> 680R
- moved D1 138.9 mm to (71.1, 79.9), turned to 180 degrees
- moved C2 128.8 mm to (71.1, 90.4), turned to 180 degrees
- moved R6 125.2 mm to (83.6, 89.7), turned to 90 degrees
- moved D2 124.5 mm to (67.3, 69.9)
- moved R4 122.1 mm to (79.8, 97.3), turned to 90 degrees
- moved C5 113.8 mm to (77.1, 71.8), turned to 90 degrees
- moved R2 112.6 mm to (90.9, 70.8), turned to 90 degrees
- moved R3 108.2 mm to (75.9, 90.1), turned to 90 degrees
- moved J5 102.4 mm to (98.8, 82.3)
- moved C1 96.4 mm to (97.8, 63.0), turned to -90 degrees
- moved R1 92.2 mm to (69.8, 63.6), turned to 180 degrees
- moved R7 85.8 mm to (125.0, 86.9), turned to -90 degrees
- moved D4 84.9 mm to (85.1, 73.8), turned to 90 degrees
- moved J4 83.3 mm to (87.4, 79.5)
- moved D5 82.6 mm to (92.7, 76.4)
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Connections:
- C1 pad 2: GND -> Net-(C1-Pad2)
- C2 pad 1: Net-(C2-Pad1) -> Net-(C1-Pad1)
- C3 pad 2: GND -> Net-(C3-Pad2)
- C4 pad 1: Net-(C2-Pad1) -> Net-(C4-Pad1)
- C4 pad 2: Net-(C4-Pad2) -> Net-(C3-Pad2)
- C5 pad 2: Net-(C5-Pad2) -> GND
- C6 pad 2: Net-(C5-Pad2) -> GND
- D1 pad 1: Net-(D1-Pad1) -> Net-(C1-Pad1)
- D1 pad 2: Net-(D1-Pad2) -> GND
- D2 pad 1: Net-(C2-Pad1) -> Net-(D1-Pad4)
- D2 pad 2: GND -> Net-(D2-Pad2)
- D3 pad 1: Net-(C1-Pad1) -> Net-(C3-Pad1)
- D3 pad 2: (no net) -> Net-(D3-Pad2)
- D4 pad 2: Net-(C4-Pad2) -> Net-(C1-Pad2)
- D5 pad 2: (no net) -> Net-(D5-Pad2)
- D6 pad 1: Net-(C5-Pad1) -> Net-(C3-Pad1)
- J4 pad 1: GND -> Net-(C5-Pad1)
- J5 pad 1: Net-(C5-Pad2) -> GND
- R1 pad 1: Net-(D1-Pad2) -> Net-(D2-Pad2)
- R1 pad 2: Net-(D2-Pad3) -> Net-(D1-Pad3)
- R2 pad 1: Net-(C3-Pad1) -> Net-(C1-Pad2)
- R3 pad 2: Net-(C2-Pad1) -> Net-(C1-Pad1)
- R5 pad 1: Net-(C4-Pad2) -> Net-(R5-Pad1)
- R5 pad 2: Net-(C2-Pad1) -> Net-(D6-Pad2)
- R6 pad 1: Net-(R6-Pad1) -> Net-(C6-Pad1)
- R6 pad 2: Net-(D6-Pad2) -> Net-(C5-Pad1)
- R7 pad 1: Net-(C5-Pad2) -> Net-(C3-Pad2)
- R7 pad 2: Net-(R6-Pad1) -> Net-(R5-Pad1)
- U1 pad 1: Net-(C3-Pad1) -> Net-(C6-Pad1)
- U2 pad 1: Net-(R4-Pad1) -> Net-(C3-Pad2)
- U2 pad 2: GND -> Net-(R5-Pad1)
- U2 pad 3: Net-(C5-Pad2) -> Net-(R4-Pad1)
- U2 pad 4: Net-(R6-Pad1) -> GND
Routing:
- net Net-(C1-Pad1): track 0.00 -> 82.8 mm
- net Net-(D4-Pad1): track 0.00 -> 56.6 mm
- net Net-(C3-Pad1): track 0.00 -> 42.8 mm
- net Net-(C4-Pad1): track 0.00 -> 37.2 mm
- net Net-(R4-Pad1): track 0.00 -> 34.6 mm
- net Net-(C5-Pad1): track 0.00 -> 22.9 mm
- net Net-(C1-Pad2): track 0.00 -> 20.2 mm
- net Net-(R5-Pad1): track 0.00 -> 16.2 mm
- net Net-(C6-Pad1): track 0.00 -> 14.0 mm
- net Net-(D1-Pad3): track 0.00 -> 12.9 mm
- net Net-(D1-Pad4): track 0.00 -> 11.6 mm
- net Net-(D3-Pad2): track 0.00 -> 9.85 mm
- net Net-(D2-Pad2): track 0.00 -> 6.35 mm
- net Net-(R3-Pad1): track 0.00 -> 6.15 mm
- net Net-(D6-Pad2): track 0.00 -> 5.46 mm
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- added copper zone on B.Cu, net GND
- added copper zone on B.Cu, net Net-(C3-Pad2)
Other:
- board outline added: 108 x 48.3 mm
