File: AC-DC Switching/AC-DC Switching.kicad_sch (KiCad schematic)
At the start: 28 parts, among them J1 AC, J2 AC, J3 12VDC, J4 0VDC, J5 DC_OUT, T1 EE22, U1 TNY267P, U2 PC817

Commit message: update folders and files
Parts:
- removed C1: 100uF/35V, Capacitor_THT:CP_Radial_D10.0mm_P5.00mm, symbol Device:CP1_Small
- removed C2: 47uF/400V, Capacitor_THT:CP_Radial_D10.0mm_P5.00mm, symbol Device:CP1_Small
- removed C5, C6: 1000uF/10V, Capacitor_THT:CP_Radial_D12.5mm_P5.00mm, symbol Device:CP1_Small
- added C2: 47u@400V, Capacitor_THT:CP_Radial_D10.0mm_P5.00mm, symbol Device:C_Polarized_Small
- added C3, C4: 1000u@10V, Capacitor_THT:CP_Radial_D12.5mm_P5.00mm, symbol Device:C_Polarized_Small
- added C5: 100u@35V, Capacitor_THT:CP_Radial_D10.0mm_P5.00mm, symbol Device:C_Polarized_Small
- added Hm1, Hm2, Hm3, Hm4: MountingHole, MountingHole:MountingHole_3.2mm_M3, symbol Mechanical:MountingHole
- C1: renamed from C4; value 2.2uF/1kV -> 2.2u@1kV
- L1: value 10uH/3A -> 10u@3A; footprint (none) -> Inductor_THT:L_Toroid_Vertical_L21.6mm_W9.1mm_P8.40mm_Bourns_5700
- R5: renamed from R6; value 59 -> 59R
- R7: value 680 -> 680R
- T1: footprint (none) -> Transformer_THT:Transformer_Myrra_EF20_7408x
- renumbered C3 to C6, D2 to D1, D1 to D2, D5 to D3, D3 to D5, J5 to J2, J2 to J3, J3 to J4, J4 to J5, R5 to R2, R2 to R6
Connections:
- net GND: now also T1.5 (SA), U2.4, C2.2, C5.2; no longer T1.3 (SA), U2.2
- net at D3.1 (K), D6.1 (K), L1.1: now also C3.1
- net at D3.2 (A): now also T1.10 (AB); no longer T1.2 (AB)
- net at R4.1, U1.4 (EN/UV): now also U2.3; no longer U2.1
- net at D4.1 (K), U1.5 (D): now also T1.2 (SC); no longer T1.5 (SC)
- net at J2.1 (Pin_1), R7.1: now also T1.8 (AA), U2.1, C3.2, C4.2; no longer T1.1 (AA), U2.3
- net at J2.2 (Pin_2), L1.2: now also C4.1
- net at C1.1, D1.1 (+), R2.2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: now also T1.1 (SD), C2.1; no longer T1.6 (SD)
- net at D5.1 (K), J4.1 (Pin_1), R6.2: now also C5.1
- net at R5.1, R7.2: now also U2.2; no longer U2.4
Other:
- moved on the sheet: C1, C6, D1, D2, D3, D4, D5, D6, J1, J2, J3, J4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
