File: Christmas tree/Christmas tree.kicad_pcb (KiCad board)
At the start: 2 copper layers, 61.2 x 77.1 mm, 14 parts, among them SW1 SWITCH

Commit message: update folders and files
Other:
- net class Default removed
