File: Christmas tree/Christmas tree.kicad_sch (KiCad schematic)
At the start: 14 parts, among them SW1 SWITCH

Commit message: update files
Other:
- company: (none) -> Cristóbal Cuevas Lagos
- title: (none) -> Christmas tree
Changed lines of the file:
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@@
 (kicad_sch (version 20211123) (generator eeschema)
-  (paper "A4")
+  (paper "USLetter")
+  (title_block
+    (title "Christmas tree")
+    (rev "1.0")
+    (company "Cristóbal Cuevas Lagos")
+  )
   (junction (at 148.844 86.614) (diameter 0) (color 0 0 0 0)
   )
