File: LED battery/DW01A.kicad_sch (KiCad schematic)
At the start: 4 parts, among them U2 DW01A

Commit message: update files
Other:
- company: (none) -> Cristóbal Cuevas Lagos
Changed lines of the file:
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@@
 (kicad_sch (version 20211123) (generator eeschema)
   (paper "A4")
+  (title_block
+    (rev "1.0")
+    (company "Cristóbal Cuevas Lagos")
+  )
   (junction (at 161.29 99.06) (diameter 0) (color 0 0 0 0)
   )
