File: LED battery/FS8205A.kicad_sch (KiCad schematic)
At the start: 1 part, among them U3 FS8205A

Commit message: update files
Other:
- company: (none) -> Cristóbal Cuevas Lagos
Changed lines of the file:
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@@
 (kicad_sch (version 20211123) (generator eeschema)
   (paper "A4")
+  (title_block
+    (rev "1.0")
+    (company "Cristóbal Cuevas Lagos")
+  )
   (junction (at 156.21 104.14) (diameter 0) (color 0 0 0 0)
   )
