File: LED circle/LED circle.kicad_sch (KiCad schematic)
At the start: 11 parts, among them Q1 BC547, SW1 EG1218

Commit message: update files
Other:
- company: (none) -> Cristóbal Cuevas Lagos
- title: (none) -> LED circle
Changed lines of the file:
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@@
 (kicad_sch (version 20211123) (generator eeschema)
   (paper "A4")
+  (title_block
+    (title "LED circle")
+    (rev "1.0")
+    (company "Cristóbal Cuevas Lagos")
+  )
   (junction (at 179.07 74.93) (diameter 0) (color 0 0 0 0)
   )
