File: LED matrix/LED matrix.kicad_sch (KiCad schematic)
At the start: 29 parts, among them J1 CONNECTOR, SW1 SWITCH, U1 ATtiny85-20PU

Commit message: update files
Other:
- company: (none) -> Cristóbal Cuevas Lagos
- title: (none) -> LED matrix
Changed lines of the file:
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@@
 (kicad_sch (version 20211123) (generator eeschema)
   (paper "A4")
+  (title_block
+    (title "LED matrix")
+    (rev "1.0")
+    (company "Cristóbal Cuevas Lagos")
+  )
   (junction (at 68.961 121.539) (diameter 0) (color 0 0 0 0)
   )
