File: PIC18F4550/PIC18F4550.kicad_pcb (KiCad board)
At the start: 2 copper layers, 100 x 70 mm, 33 parts, among them J1 PORT_D, J10 USB_B, J11 PICKIT, J2 PORT_A, J3 PORT_E, J4 PORT_B, J5 PORT_C, J6 GND, J7 VOL, J8 VOLT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

Commit message: update files
Other:
- net class Default removed
