File: Panel 7 segments/Panel 7 segments.kicad_sch (KiCad schematic)
At the start: 41 parts, among them J1 ENTRADA, J2 SALIDA, U1 STP16CP05, U2 AMS1117-3.3

Commit message: update files
Other:
- company: (none) -> Cristóbal Cuevas Lagos
- title: (none) -> Panel 7 segments
Changed lines of the file:
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@@
 (kicad_sch (version 20211123) (generator eeschema)
   (paper "USLetter")
+  (title_block
+    (title "Panel 7 segments")
+    (rev "1.0")
+    (company "Cristóbal Cuevas Lagos")
+    (comment 1 "Large 7 segment panel controlled by STP16CP05 IC and allows connecting several in series")
+  )
   (junction (at 222.25 73.66) (diameter 0) (color 0 0 0 0)
   )
