File: STM32F030/STM32F030.kicad_sch (KiCad schematic)
At the start: 14 parts, among them J1 Connector, J2 USB_B_Micro, U1 STM32F030, U2 LD1117S33TR_SOT223

Commit message: update files
Other:
- company: (none) -> Cristóbal Cuevas Lagos
- title: Programación STM32 -> STM32F030
Changed lines of the file:
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@@
   (paper "USLetter")
   (title_block
-    (title "Programación STM32")
+    (title "STM32F030")
     (date "2020-08-21")
+    (rev "1.0")
+    (company "Cristóbal Cuevas Lagos")
+    (comment 1 "Basic programmer for STM32F0")
   )
   (junction (at 158.496 127) (diameter 0) (color 0 0 0 0)
