File: USB to UART/CP2102N-GQFN28.kicad_sch (KiCad schematic)
At the start: 10 parts, among them U1 CP2102N-A01-GQFN28

Commit message: update files
Other:
- company: (none) -> Cristóbal Cuevas Lagos
- title: (none) -> CP2102N
Changed lines of the file:
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@@
   (paper "USLetter")
   (title_block
-    (date "2021-06-15")
+    (title "CP2102N")
+    (rev "1.0")
+    (company "Cristóbal Cuevas Lagos")
+    (comment 1 "Cristóbal Cuevas Lagos")
   )
   (junction (at 44.45 97.79) (diameter 0) (color 0 0 0 0)
