File: USB to UART/Connector.kicad_sch (KiCad schematic)
At the start: 1 part, among them J1 Connectors

Commit message: update files
Other:
- company: (none) -> Cristóbal Cuevas Lagos
- title: (none) -> Connector
Changed lines of the file:
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@@
   (paper "USLetter")
   (title_block
-    (date "2021-06-15")
+    (title "Connector")
+    (rev "1.0")
+    (company "Cristóbal Cuevas Lagos")
+    (comment 1 "Cristóbal Cuevas Lagos")
   )
   (wire (pts (xy 132.08 100.33) (xy 137.16 100.33))
