File: USB to UART/USB to UART.kicad_pcb (KiCad board)
At the start: 2 copper layers, 39.4 x 19 mm, 14 parts, among them J1 Connectors, J2 USB_A, U1 CP2102N-A01-GQFN28

Commit message: update schematics
Parts:
- C1, C2, C3, C4: footprint Capacitor_SMD:C_1206_3216Metric -> Capacitor_SMD:C_0603_1608Metric
- D1, D2, D3: footprint LED_SMD:LED_1206_3216Metric -> LED_SMD:LED_0603_1608Metric
- R1, R2, R3, R4: footprint Resistor_SMD:R_1206_3216Metric -> Resistor_SMD:R_0603_1608Metric
- moved R4 10.1 mm to (146.4, 118.9)
- moved C1 6.79 mm to (150.7, 119.4)
- moved D3 5.90 mm to (146.3, 117.3)
- moved C2 5.90 mm to (152.3, 119.4)
- moved D1 3.36 mm to (162.8, 118.6), turned to 0 degrees
- moved R3 3.28 mm to (162.0, 112.8), turned to -90 degrees
- moved D2 2.45 mm to (162.8, 109.9), turned to 0 degrees
- moved C4 2.32 mm to (153.9, 119.4)
- moved R2 2.29 mm to (162.0, 115.9), turned to 90 degrees
- moved C3 1.45 mm to (155.5, 119.4)
- moved R1 0.53 mm to (157.0, 119.4)
Connections:
- net /Alimentacion/D+ renamed /CP2102N-GQFN28/D+
- net /Alimentacion/D- renamed /CP2102N-GQFN28/D-
- net /CP2102N-GQFN28/+5V renamed /USB/POWER
- net /CP2102N-GQFN28/RXD renamed /CP2102N-GQFN28/RX
- net /CP2102N-GQFN28/TXD renamed /CP2102N-GQFN28/TX
- U1 pad 1: (no net) -> unconnected-(U1-Pad1)
- U1 pad 10: (no net) -> unconnected-(U1-Pad10)
- U1 pad 11: (no net) -> unconnected-(U1-Pad11)
- U1 pad 12: (no net) -> unconnected-(U1-Pad12)
- U1 pad 13: (no net) -> unconnected-(U1-Pad13)
- U1 pad 14: (no net) -> unconnected-(U1-Pad14)
- U1 pad 15: (no net) -> unconnected-(U1-Pad15)
- U1 pad 16: (no net) -> unconnected-(U1-Pad16)
- U1 pad 17: (no net) -> unconnected-(U1-Pad17)
- U1 pad 18: (no net) -> unconnected-(U1-Pad18)
- U1 pad 19: (no net) -> unconnected-(U1-Pad19)
- U1 pad 2: (no net) -> unconnected-(U1-Pad2)
- U1 pad 20: (no net) -> unconnected-(U1-Pad20)
- U1 pad 21: (no net) -> unconnected-(U1-Pad21)
- U1 pad 22: (no net) -> unconnected-(U1-Pad22)
- U1 pad 23: (no net) -> unconnected-(U1-Pad23)
- U1 pad 24: (no net) -> unconnected-(U1-Pad24)
- U1 pad 27: (no net) -> unconnected-(U1-Pad27)
Routing:
- net /CP2102N-GQFN28/3V3: track 33.2 -> 19.7 mm
- net GND: track 12.4 -> 9.40 mm, vias 5 -> 4
- net /USB/POWER: track 20.8 -> 22.4 mm, vias 2 -> 0
- net Net-(D2-Pad1): track 2.69 -> 1.79 mm
- net Net-(D1-Pad1): track 2.76 -> 1.91 mm
- net /CP2102N-GQFN28/TX: track 20.1 -> 19.2 mm, vias 1 -> 0
- net Net-(D3-Pad2): track 2.44 -> 1.68 mm
- net Net-(R1-Pad2): track 4.64 -> 5.21 mm
