File: USB to UART/USB to UART.kicad_sch (KiCad schematic)
At the start: 0 parts

Commit message: update folders and files
Other:
- sheet Alimentacion renamed Source
- sheet Source: file Alimentacion.kicad_sch -> Source.kicad_sch
Changed lines of the file:
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@@
     (stroke (width 0) (type solid) (color 0 0 0 0))
     (fill (color 0 0 0 0.0000))
-    (property "Sheet name" "Alimentacion" (id 0) (at 93.98 86.9184 0)
+    (property "Sheet name" "Source" (id 0) (at 93.98 86.9184 0)
       (effects (font (size 1.27 1.27)) (justify left bottom))
     )
-    (property "Sheet file" "Alimentacion.kicad_sch" (id 1) (at 93.98 100.9146 0)
+    (property "Sheet file" "Source.kicad_sch" (id 1) (at 93.98 100.9146 0)
       (effects (font (size 1.27 1.27)) (justify left top))
     )

Commit message: update files
Other:
- sheet Source renamed USB
- sheet USB: file Source.kicad_sch -> USB.kicad_sch
- company: (none) -> Cristóbal Cuevas Lagos
- title: (none) -> USB  to UART
Changed lines of the file:
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@@
 (kicad_sch (version 20211123) (generator eeschema)
-  (paper "A4")
-  (wire (pts (xy 205.74 101.6) (xy 205.74 102.87))
+  (paper "USLetter")
+  (title_block
+    (title "USB  to UART")
+    (rev "1.0")
+    (company "Cristóbal Cuevas Lagos")
+    (comment 1 "USB to UART converter with CP2102 IC")
+  )
+  (wire (pts (xy 196.85 103.505) (xy 196.85 104.775))
     (stroke (width 0) (type default) (color 0 0 0 0))
   )
-  (wire (pts (xy 91.44 96.52) (xy 93.98 96.52))
+  (wire (pts (xy 82.55 98.425) (xy 85.09 98.425))
     (stroke (width 0) (type default) (color 0 0 0 0))
   )
-  (wire (pts (xy 201.93 101.6) (xy 205.74 101.6))
+  (wire (pts (xy 193.04 103.505) (xy 196.85 103.505))
     (stroke (width 0) (type default) (color 0 0 0 0))
   )
-  (wire (pts (xy 130.81 102.87) (xy 130.81 101.6))
+  (wire (pts (xy 121.92 104.775) (xy 121.92 103.505))
     (stroke (width 0) (type default) (color 0 0 0 0))
   )
-  (wire (pts (xy 165.1 96.52) (xy 177.8 96.52))
+  (wire (pts (xy 156.21 98.425) (xy 168.91 98.425))
     (stroke (width 0) (type default) (color 0 0 0 0))
   )
-  (wire (pts (xy 120.65 91.44) (xy 133.35 91.44))
+  (wire (pts (xy 111.76 93.345) (xy 124.46 93.345))
     (stroke (width 0) (type default) (color 0 0 0 0))
   )
-  (wire (pts (xy 130.81 101.6) (xy 133.35 101.6))
+  (wire (pts (xy 121.92 103.505) (xy 124.46 103.505))
     (stroke (width 0) (type default) (color 0 0 0 0))
   )
-  (wire (pts (xy 120.65 93.98) (xy 133.35 93.98))
+  (wire (pts (xy 111.76 95.885) (xy 124.46 95.885))
     (stroke (width 0) (type default) (color 0 0 0 0))
   )
-  (wire (pts (xy 165.1 99.06) (xy 177.8 99.06))
+  (wire (pts (xy 156.21 100.965) (xy 168.91 100.965))
     (stroke (width 0) (type default) (color 0 0 0 0))
   )
-  (wire (pts (xy 165.1 93.98) (xy 177.8 93.98))
+  (wire (pts (xy 156.21 95.885) (xy 168.91 95.885))
     (stroke (width 0) (type default) (color 0 0 0 0))
   )
-  (wire (pts (xy 91.44 97.79) (xy 91.44 96.52))
+  (wire (pts (xy 82.55 99.695) (xy 82.55 98.425))
     (stroke (width 0) (type default) (color 0 0 0 0))
   )
-  (wire (pts (xy 120.65 96.52) (xy 133.35 96.52))
+  (wire (pts (xy 111.76 98.425) (xy 124.46 98.425))
     (stroke (width 0) (type default) (color 0 0 0 0))
   )
-  (wire (pts (xy 165.1 101.6) (xy 177.8 101.6))
+  (wire (pts (xy 156.21 103.505) (xy 168.91 103.505))
     (stroke (width 0) (type default) (color 0 0 0 0))
   )
-  (wire (pts (xy 165.1 91.44) (xy 177.8 91.44))
+  (wire (pts (xy 156.21 93.345) (xy 168.91 93.345))
     (stroke (width 0) (type default) (color 0 0 0 0))
   )
-  (symbol (lib_id "power:GND") (at 205.74 102.87 0) (unit 1)
+  (symbol (lib_id "power:GND") (at 196.85 104.775 0) (unit 1)
     (in_bom yes) (on_board yes)
-    (property "Reference" "#PWR0101" (id 0) (at 205.74 109.22 0)
+    (property "Reference" "#PWR0101" (id 0) (at 196.85 111.125 0)
       (effects (font (size 1.27 1.27)) hide)
     )
-    (property "Value" "GND" (id 1) (at 205.867 107.2642 0))
-    (property "Footprint" "" (id 2) (at 205.74 102.87 0)
+    (property "Value" "GND" (id 1) (at 196.977 109.1692 0))
+    (property "Footprint" "" (id 2) (at 196.85 104.775 0)
       (effects (font (size 1.27 1.27)) hide)
     )
-    (property "Datasheet" "" (id 3) (at 205.74 102.87 0)
+    (property "Datasheet" "" (id 3) (at 196.85 104.775 0)
       (effects (font (size 1.27 1.27)) hide)
     )
     (pin "1")
   )
-  (symbol (lib_id "power:GND") (at 130.81 102.87 0) (unit 1)
+  (symbol (lib_id "power:GND") (at 121.92 104.775 0) (unit 1)
     (in_bom yes) (on_board yes)
-    (property "Reference" "#PWR0102" (id 0) (at 130.81 109.22 0)
+    (property "Reference" "#PWR0102" (id 0) (at 121.92 111.125 0)
       (effects (font (size 1.27 1.27)) hide)
     )
-    (property "Value" "GND" (id 1) (at 130.937 107.2642 0))
-    (property "Footprint" "" (id 2) (at 130.81 102.87 0)
+    (property "Value" "GND" (id 1) (at 122.047 109.1692 0))
+    (property "Footprint" "" (id 2) (at 121.92 104.775 0)
       (effects (font (size 1.27 1.27)) hide)
     )
-    (property "Datasheet" "" (id 3) (at 130.81 102.87 0)
+    (property "Datasheet" "" (id 3) (at 121.92 104.775 0)
       (effects (font (size 1.27 1.27)) hide)
     )
     (pin "1")
   )
-  (symbol (lib_id "power:GND") (at 91.44 97.79 0) (unit 1)
+  (symbol (lib_id "power:GND") (at 82.55 99.695 0) (unit 1)
     (in_bom yes) (on_board yes)
-    (property "Reference" "#PWR0103" (id 0) (at 91.44 104.14 0)
+    (property "Reference" "#PWR0103" (id 0) (at 82.55 106.045 0)
       (effects (font (size 1.27 1.27)) hide)
     )
-    (property "Value" "GND" (id 1) (at 91.567 102.1842 0))
-    (property "Footprint" "" (id 2) (at 91.44 97.79 0)
+    (property "Value" "GND" (id 1) (at 82.677 104.0892 0))
+    (property "Footprint" "" (id 2) (at 82.55 99.695 0)
       (effects (font (size 1.27 1.27)) hide)
     )
-    (property "Datasheet" "" (id 3) (at 91.44 97.79 0)
+    (property "Datasheet" "" (id 3) (at 82.55 99.695 0)
       (effects (font (size 1.27 1.27)) hide)
     )
     (pin "1")
   )
-  (sheet (at 133.35 87.63) (size 31.75 17.78) (fields_autoplaced)
+  (sheet (at 124.46 89.535) (size 31.75 17.78) (fields_autoplaced)
     (stroke (width 0) (type solid) (color 0 0 0 0))
     (fill (color 0 0 0 0.0000))
-    (property "Sheet name" "CP2102N-GQFN28" (id 0) (at 133.35 86.9184 0)
+    (property "Sheet name" "CP2102N-GQFN28" (id 0) (at 124.46 88.8234 0)
       (effects (font (size 1.27 1.27)) (justify left bottom))
     )
-    (property "Sheet file" "CP2102N-GQFN28.kicad_sch" (id 1) (at 133.35 105.9946 0)
+    (property "Sheet file" "CP2102N-GQFN28.kicad_sch" (id 1) (at 124.46 107.8996 0)
       (effects (font (size 1.27 1.27)) (justify left top))
     )
-    (pin "TXD" output (at 165.1 96.52 0)
+    (pin "TXD" output (at 156.21 98.425 0)
       (effects (font (size 1.27 1.27)) (justify right))
     )
-    (pin "RXD" input (at 165.1 93.98 0)
+    (pin "RXD" input (at 156.21 95.885 0)
       (effects (font (size 1.27 1.27)) (justify right))
     )
-    (pin "DTR" output (at 165.1 91.44 0)
+    (pin "DTR" output (at 156.21 93.345 0)
       (effects (font (size 1.27 1.27)) (justify right))
     )
-    (pin "D+" input (at 133.35 93.98 180)
+    (pin "D+" input (at 124.46 95.885 180)
       (effects (font (size 1.27 1.27)) (justify left))
     )
-    (pin "D-" input (at 133.35 96.52 180)
+    (pin "D-" input (at 124.46 98.425 180)
       (effects (font (size 1.27 1.27)) (justify left))
     )
-    (pin "VBUS" input (at 133.35 91.44 180)
+    (pin "VBUS" input (at 124.46 93.345 180)
       (effects (font (size 1.27 1.27)) (justify left))
     )
-    (pin "GND" input (at 133.35 101.6 180)
+    (pin "GND" input (at 124.46 103.505 180)
       (effects (font (size 1.27 1.27)) (justify left))
     )
-    (pin "3V3" output (at 165.1 101.6 0)
+    (pin "3V3" output (at 156.21 103.505 0)
       (effects (font (size 1.27 1.27)) (justify right))
     )
-    (pin "+5V" output (at 165.1 99.06 0)
+    (pin "+5V" output (at 156.21 100.965 0)
       (effects (font (size 1.27 1.27)) (justify right))
     )
   )
-  (sheet (at 177.8 87.63) (size 24.13 17.78) (fields_autoplaced)
+  (sheet (at 168.91 89.535) (size 24.13 17.78) (fields_autoplaced)
     (stroke (width 0) (type solid) (color 0 0 0 0))
     (fill (color 0 0 0 0.0000))
-    (property "Sheet name" "Connector" (id 0) (at 177.8 86.9184 0)
+    (property "Sheet name" "Connector" (id 0) (at 168.91 88.8234 0)
       (effects (font (size 1.27 1.27)) (justify left bottom))
     )
-    (property "Sheet file" "Connector.kicad_sch" (id 1) (at 177.8 105.9946 0)
+    (property "Sheet file" "Connector.kicad_sch" (id 1) (at 168.91 107.8996 0)
       (effects (font (size 1.27 1.27)) (justify left top))
     )
-    (pin "DTR" input (at 177.8 91.44 180)
+    (pin "DTR" input (at 168.91 93.345 180)
       (effects (font (size 1.27 1.27)) (justify left))
     )
-    (pin "RXD" output (at 177.8 93.98 180)
+    (pin "RXD" output (at 168.91 95.885 180)
       (effects (font (size 1.27 1.27)) (justify left))
     )
-    (pin "TXD" input (at 177.8 96.52 180)
+    (pin "TXD" input (at 168.91 98.425 180)
       (effects (font (size 1.27 1.27)) (justify left))
     )
-    (pin "+5V" input (at 177.8 99.06 180)
+    (pin "+5V" input (at 168.91 100.965 180)
       (effects (font (size 1.27 1.27)) (justify left))
     )
-    (pin "GND" output (at 201.93 101.6 0)
+    (pin "GND" output (at 193.04 103.505 0)
       (effects (font (size 1.27 1.27)) (justify right))
     )
-    (pin "3V3" input (at 177.8 101.6 180)
+    (pin "3V3" input (at 168.91 103.505 180)
       (effects (font (size 1.27 1.27)) (justify left))
     )
   )
-  (sheet (at 93.98 87.63) (size 26.67 12.7) (fields_autoplaced)
+  (sheet (at 85.09 89.535) (size 26.67 12.7) (fields_autoplaced)
     (stroke (width 0) (type solid) (color 0 0 0 0))
     (fill (color 0 0 0 0.0000))
-    (property "Sheet name" "Source" (id 0) (at 93.98 86.9184 0)
+    (property "Sheet name" "USB" (id 0) (at 85.09 88.8234 0)
       (effects (font (size 1.27 1.27)) (justify left bottom))
     )
-    (property "Sheet file" "Source.kicad_sch" (id 1) (at 93.98 100.9146 0)
+    (property "Sheet file" "USB.kicad_sch" (id 1) (at 85.09 102.8196 0)
       (effects (font (size 1.27 1.27)) (justify left top))
     )
-    (pin "VBUS" input (at 120.65 91.44 0)
+    (pin "VBUS" input (at 111.76 93.345 0)
       (effects (font (size 1.27 1.27)) (justify right))
     )
-    (pin "D+" input (at 120.65 93.98 0)
+    (pin "D+" input (at 111.76 95.885 0)
       (effects (font (size 1.27 1.27)) (justify right))
     )
-    (pin "D-" input (at 120.65 96.52 0)
+    (pin "D-" input (at 111.76 98.425 0)
       (effects (font (size 1.27 1.27)) (justify right))
     )
-    (pin "GND" output (at 93.98 96.52 180)
+    (pin "GND" output (at 85.09 98.425 180)
       (effects (font (size 1.27 1.27)) (justify left))
     )

Commit message: update schematics
Parts:
- added C? (x2): 4.7u, Capacitor_SMD:C_0603_1608Metric, symbol Device:C_Small
- added C? (x2): 0.1u, Capacitor_SMD:C_0603_1608Metric, symbol Device:C_Small
- added D?: LED_POWER, LED_SMD:LED_0603_1608Metric, symbol Device:LED_Small
- added D?: LED_TX, LED_SMD:LED_0603_1608Metric, symbol Device:LED_Small
- added D?: LED_RX, LED_SMD:LED_0603_1608Metric, symbol Device:LED_Small
- added J?: USB_A, USB to UART:CONECTOR USB, symbol Connector:USB_A
- added J?: Connectors, Connector_PinHeader_2.54mm:PinHeader_1x06_P2.54mm_Horizontal, symbol Connector_Generic:Conn_01x06
- added R?: 1k, Resistor_SMD:R_0603_1608Metric, symbol Device:R_Small
- added R? (x3): 220, Resistor_SMD:R_0603_1608Metric, symbol Device:R_Small
- added U?: CP2102N-A01-GQFN28, Package_DFN_QFN:QFN-28-1EP_5x5mm_P0.5mm_EP3.35x3.35mm, symbol Interface_USB:CP2102N-A01-GQFN28
Connections:
- net GND: now also C?.1, C?.1, C?.2, C?.2, D?.1 (K), J?.4 (GND), J?.5 (Pin_5), J?.5 (Shield), U?.29 (GND), U?.3 (GND)
- new net: R?.2, U?.9 (~{RSTb})
- new net: D?.2 (A), R?.2
- new net: D?.1 (K), R?.1 (x2)
- new net +5V: C?.1, C?.2, D?.2 (A), D?.2 (A), J?.1 (VBUS), J?.4 (Pin_4), R?.1, U?.7 (REGIN), U?.8 (VBUS)
- new net 3V3: C?.1, C?.2, J?.6 (Pin_6), R?.1, U?.6 (VDD)
- new net D+: J?.3 (D+), U?.4 (D+)
- new net D-: J?.2 (D-), U?.5 (D-)
- new net DTR: J?.1 (Pin_1), U?.28 (~{DTR})
- new net RXD: J?.2 (Pin_2), R?.2, U?.25 (RXD)
- new net TXD: J?.3 (Pin_3), R?.2, U?.26 (TXD)
- no-connect marks 0 -> 17
Other:
- removed sheet CP2102N-GQFN28
- removed sheet Connector
- removed sheet USB
