File: DS3231/DS3231.kicad_sch (KiCad schematic)
At the start: 4 parts

Commit message: update projects
Parts:
- added D1: 1N4148, Diode_THT:D_DO-35_SOD27_P7.62mm_Horizontal, symbol Diode:1N4148
- added J1: Conn_01x06, Connector_PinHeader_2.54mm:PinHeader_1x06_P2.54mm_Vertical_SMD_Pin1Left, symbol Connector_Generic:Conn_01x06
- added J3: Conn_01x04, Connector_PinHeader_2.54mm:PinHeader_1x04_P2.54mm_Vertical_SMD_Pin1Left, symbol Connector_Generic:Conn_01x04
- added R1: 200R, Resistor_SMD:R_0805_2012Metric, symbol Device:R_Small
- added RN1: 4k7, Resistor_SMD:R_Array_Concave_4x0603, symbol Device:R_Pack04
- C1: renamed from C?; value C_Small -> 0.1u; footprint (none) -> Capacitor_SMD:C_0805_2012Metric
- C2: renamed from C?; value C_Small -> 1u; footprint (none) -> Capacitor_SMD:C_0805_2012Metric
- J2: renamed from J?; value BATTERY -> BATTERY 2032
- gave numbers to parts that had none: 1
Connections:
- net GND: now also J1.6 (Pin_6), J3.4 (Pin_4)
- net VBAT: now also D1.1 (K)
- net VCC: now also J1.5 (Pin_5), J3.3 (Pin_3), R1.1, RN1.5 (R4.2), RN1.6 (R3.2), RN1.7 (R2.2), RN1.8 (R1.2)
- net 32K: now reaches U1.1 (32KHZ)
- net 32K: now also J1.1 (Pin_1), RN1.3 (R3.1)
- net SDA: now reaches U1.15 (SDA)
- net SDA: now also J1.4 (Pin_4), J3.2 (Pin_2), RN1.2 (R2.1)
- net SCL: now reaches U1.16 (SCL)
- net SCL: now also J1.3 (Pin_3), J3.1 (Pin_1), RN1.1 (R1.1)
- net SQW: now reaches U1.3 (~{INT}/SQW)
- net SQW: now also J1.2 (Pin_2), RN1.4 (R4.1)
- new net: D1.2 (A), R1.2
- no-connect marks 0 -> 1
Other:
- note added: "I2C Adress: 0x68"
- note added: "Supply Voltage: 2.3 to 5.5"
- company: (none) -> Cristóbal Cuevas Lagos
- title: (none) -> DS3231
- moved on the sheet: C1, C2, J2, U1
