File: PROYECTO/PROYECTO.kicad_pcb (KiCad board)
At the start: 2 copper layers, 52 parts, among them J1 Conn_01x08, J2 Conn_01x03, J3 Conn_01x05, J4 Conn_01x05, J5 Conn_01x04, Q1 2N2222, U1 TL062, U2 TL062, U3 TL062, U4 TL062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

Commit message: update schematics
Parts:
- moved J1 98.6 mm to (107.2, 134.1)
- moved R15 81.5 mm to (178.1, 116.9), turned to 0 degrees
- moved RV4 80.3 mm to (184.4, 129.0)
- moved R10 79.8 mm to (127.0, 121.7), turned to 90 degrees
- moved RV5 76.4 mm to (94.1, 129.0)
- moved J2 75.9 mm to (168.1, 129.0)
- moved R11 75.5 mm to (110.2, 118.7)
- moved R8 75.4 mm to (99.7, 106.2)
- moved RV2 75.2 mm to (87.9, 129.0), turned to -90 degrees
- moved R13 75.1 mm to (110.2, 113.6)
- moved R3 75.0 mm to (131.1, 114.2), turned to -90 degrees
- moved U1 75.0 mm to (134.9, 114.2)
- moved U3 75.0 mm to (167.4, 111.9)
- moved RV3 75.0 mm to (124.6, 106.1)
- moved U2 75.0 mm to (92.1, 111.0)
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Routing:
- net Net-(R1-Pad1): track 0.00 -> 30.4 mm
- net /PID/SP: track 7.86 -> 26.5 mm
- net /PID/ERROR: track 28.3 -> 11.3 mm
- net Net-(R5-Pad2): track 21.5 -> 37.6 mm
- net Net-(R3-Pad2): track 0.00 -> 14.3 mm
- net /PID/INTEGRAL: track 20.7 -> 34.4 mm
- net /PID/PROPORCIONAL: track 11.1 -> 23.5 mm
- net VEE: track 0.00 -> 12.2 mm
- net Net-(R13-Pad1): track 18.4 -> 30.5 mm
- net Net-(R14-Pad1): track 6.94 -> 17.8 mm
- net OUT: track 8.78 -> 18.2 mm
- net Net-(C1-Pad1): track 17.3 -> 26.4 mm
- net /PID/PERTURBACIÓN: track 15.4 -> 7.16 mm
- net Net-(R10-Pad2): track 0.00 -> 8.04 mm
- net GV+: track 44.1 -> 36.1 mm
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Other:
- board outline added: 111.8 x 76.2 mm
