File: STM32F103/STM32F103.kicad_pcb (KiCad board)
At the start: 4 copper layers, 28 parts, among them J1 USB_B_Micro, J2 Conn_01x15, J3 Conn_01x15, U1 XC6206PxxxMR, U2 USBLC6-2SC6, U3 STM32F103CBTx, Y1 8MHz

Commit message: update schematics
Parts:
- moved R1 24.1 mm to (156.9, 109.9)
- moved C1 24.0 mm to (150.2, 109.2)
- moved FB1 24.0 mm to (150.2, 105.4)
- moved C8 24.0 mm to (130.6, 101.0)
- moved R3 24.0 mm to (128.1, 106.2)
- moved R4 24.0 mm to (147.0, 98.1)
- moved B0 24.0 mm to (137.3, 89.4)
- moved J1 24.0 mm to (159.4, 98.7)
- moved J2 24.0 mm to (158.1, 85.1)
- moved U3 24.0 mm to (138.1, 100.0)
- moved Y1 24.0 mm to (127.3, 99.4)
- moved C10 24.0 mm to (127.3, 95.5)
- moved C11 24.0 mm to (127.3, 103.3)
- moved C2 24.0 mm to (154.9, 106.2)
- moved C3 24.0 mm to (133.2, 93.7)
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Routing:
- net unconnected-(J1-Pad6): track 0.00 -> 15.2 mm
- net +3V3: track 10.4 -> 12.5 mm
- net GND: track 31.7 -> 30.2 mm, vias 15 -> 16
Other:
- board outline added: 42.7 x 34.5 mm
- copper layers 4 -> 2
