File: SX1276/SX1276 IC.kicad_sch (KiCad schematic)
At the start: 19 parts

Commit message: update schematics
Parts:
- removed C? (x6): C_Small, symbol Device:C_Small
- removed C? (x5): 100n, symbol Device:C_Small
- removed C?: 1u, symbol Device:C_Small
- removed JP?: VDD_RFS, symbol Jumper:Jumper_2_Bridged
- removed R? (x2): 0R, symbol Device:R_Small
- removed TP?: RXTX_RF, symbol Connector:TestPoint
- removed TP?: GND, symbol Connector:TestPoint
- removed U?: SX1276, Package_DFN_QFN:QFN-28-1EP_6x6mm_P0.65mm_EP4.8x4.8mm, symbol RF:SX1276
- removed Y?: 32MHz, symbol Device:Crystal_GND24
- added C1, C15: 1nF, Capacitors_SMD:C_0402, symbol lora-module-rescue:C
- added C10, C14: 3.3pF, Capacitors_SMD:C_0402, symbol lora-module-rescue:C
- added C11, C13, C21, C4, C7: 47pF, Capacitors_SMD:C_0402, symbol lora-module-rescue:C
- added C12, C18, C19, C20, C22: 100nF, Capacitors_SMD:C_0402, symbol lora-module-rescue:C
- added C16, C17: 15pF, Capacitors_SMD:C_0402, symbol lora-module-rescue:C
- added C2: 10uF, Capacitors_SMD:C_0805, symbol lora-module-rescue:C
- added C3: 10nF, Capacitors_SMD:C_0402, symbol lora-module-rescue:C
- added C5: 1.5pF, Capacitors_SMD:C_0402, symbol lora-module-rescue:C
- added C6: 22pF, Capacitors_SMD:C_0402, symbol lora-module-rescue:C
- added C8, C9: 8.2pF, Capacitors_SMD:C_0402, symbol lora-module-rescue:C
- added J1: SMA, balcerzak-pcb:SMA-16, symbol lora-module-rescue:CONN_COAXIAL
- added L1: 33nH Wire, Inductors_SMD:L_0402, symbol lora-module-rescue:INDUCTOR
- added L2: 2.2nH Wire, Inductors_SMD:L_0402, symbol lora-module-rescue:INDUCTOR
- added L3: 5.6nH Wire, Inductors_SMD:L_0402, symbol lora-module-rescue:INDUCTOR
- added L4: 4.7nH Wire, Inductors_SMD:L_0402, symbol lora-module-rescue:INDUCTOR
- added L5: 0R, Inductors_SMD:L_0402, symbol lora-module-rescue:INDUCTOR
- added L6: 10nH Wire, Inductors_SMD:L_0402, symbol lora-module-rescue:INDUCTOR
- added P1, P2: CONN_01X07, Pin_Headers:Pin_Header_Straight_1x07_Pitch2.54mm, symbol lora-module-rescue:CONN_01X07
- added Q1: 32MHz, Crystals:Crystal_SMD_EuroQuartz_MT-4pin_3.2x2.5mm, symbol lora-module-rescue:CRYSTAL_SMD
- added R1: 1k, Resistors_SMD:R_0402, symbol lora-module-rescue:R
- added SH1: RF_Shield_One_Piece, balcerzak-pcb:inAIR9B_shield, symbol lora-module-rescue:RF_Shield_One_Piece
- added U1: PE4259, balcerzak-pcb:SOT-363_SC-70-6, symbol lora-module-rescue:PE4259
- added U2: SX1276, Housings_DFN_QFN:QFN-28-1EP_6x6mm_Pitch0.65mm, symbol lora-module-rescue:SX1276
Connections:
- net DIO0: now also P1.5 (P5), U2.8 (DIO0)
- net DIO1: now also P1.6 (P6), U2.9 (DIO1)
- net DIO2: now also P1.7 (P7), U2.10 (DIO2)
- net DIO3: now also P1.3 (P3), U2.11 (DIO3)
- net GND: now also C1.1, C10.1, C11.2, C12.2, C14.2, C15.1, C16.2, C17.2, C18.2, C19.2, C2.2, C20.2, C21.2, C22.2, C3.2, C4.2, C8.2, C9.2, J1.2 (Ext), P1.1 (P1), Q1.2 (case), SH1.1 (Shield), U1.2 (GND), U2.15 (GND), U2.23 (GND), U2.26 (GND), U2.29 (GND)
- net MISO: now also P2.4 (P4), U2.17 (MISO)
- net MOSI: now also P2.5 (P5), U2.18 (MOSI)
- new net: C5.2, C9.1, L3.2, L4.1
- new net: C10.2, C5.1, L4.2, U1.1 (RF1)
- new net: C17.1, Q1.3, U2.5 (XTA)
- new net: C3.1, C4.1, L1.1, U2.25 (VR_PA)
- new net: C15.2, R1.1, U1.4 (CTRL)
- new net: C7.1, L5.1
- new net: C7.2, U1.5 (RFC)
- new net: C18.1, U2.2 (VR_ANA)
- new net: R1.2, U2.20 (RXTX/RFMOD)
- new net: L6.1, U2.21 (RFI_HF)
- new net: L2.1, U2.27 (PA_BOOST)
- new net: C19.1, U2.4 (VR_DIG)
- new net: C16.1, Q1.1, U2.6 (XTB)
- new net: C6.2, C8.1, L1.2, L2.2
- new net: C13.2, C14.1, L6.2
- new net: C6.1, L3.1
- new net: J1.1 (In), L5.2
- new net: C13.1, U1.3 (RF2)
- new net +3V3: C1.2, C11.1, C12.1, C2.1, C20.1, C21.1, C22.1, P2.2 (P2), U1.6 (VCC), U2.14 (VBAT_DIG), U2.24 (VBAT_RF), U2.3 (VBAT_ANA)
- new net CLK: P2.3 (P3), U2.16 (SCK)
- new net CS: P1.2 (P2), U2.19 (NSS)
- new net RST: P1.4 (P4), U2.7 (NRESET)
- no-connect marks 1 -> 7
Other:
- company: (none) -> Cristóbal Cuevas Lagos
- title: (none) -> SX1276
