File: Mixed signal/Mixed signal.kicad_pcb (KiCad board)
At the start: 2 copper layers, 114 parts, among them J200 USB_C_Receptacle_USB2.0, J201 2x5 1.27mm, J300 031-5640-1010, J400 031-5640-1010, U100 HT7533-1, U101 TLV62569DBV, U102 MCP6001T-E/OT, U200 STM32F103CBT6, U201 USBLC6-2SC6, U300 MCP6001T-E/OT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

Commit message: update schematics
Parts:
- moved J300 162.8 mm to (102.6, 177.9), turned to 180 degrees
- moved J400 158.0 mm to (146.3, 177.9), turned to 180 degrees
- moved U303 129.3 mm to (105.7, 126.0)
- moved U300 125.1 mm to (101.6, 158.5)
- moved C302 122.5 mm to (99.1, 150.4)
- moved C308 121.5 mm to (98.6, 135.1), turned to 180 degrees
- moved C306 120.5 mm to (114.8, 152.4)
- moved C311 118.6 mm to (103.1, 127.5), turned to 90 degrees
- moved C309 115.5 mm to (98.6, 133.1), turned to 180 degrees
- moved U301 113.4 mm to (115.8, 159.0)
- moved H1 112.8 mm to (71.8, -0.06)
- moved H2 112.8 mm to (79.8, 7.89)
- moved H3 112.8 mm to (71.8, 7.89)
- moved H4 112.8 mm to (79.8, -0.06)
- moved R308 112.0 mm to (101.1, 134.1), turned to -90 degrees
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Other:
- copper layers 2 -> 4

Commit message: update mixed signal
Parts:
- moved H2 149.5 mm to (164.0, 131.5)
- moved H3 130.6 mm to (114.0, 131.5)
- moved U400 113.0 mm to (149.2, 104.6)
- moved H4 107.3 mm to (164.0, 66.5)
- moved R305 86.2 mm to (123.6, 113.2)
- moved C303 85.6 mm to (126.2, 114.7), turned to -90 degrees
- moved R304 83.0 mm to (125.2, 113.7), turned to -90 degrees
- moved L101 82.5 mm to (155.1, 69.5)
- moved R301 81.1 mm to (129.7, 115.7), turned to -90 degrees
- moved R303 80.2 mm to (127.7, 114.2)
- moved D300 80.1 mm to (128.5, 119.5)
- moved C301 79.9 mm to (132.8, 115.7), turned to 180 degrees
- moved C305 79.2 mm to (126.7, 113.2)
- moved H1 78.8 mm to (114.0, 66.5)
- moved R302 77.8 mm to (132.8, 114.7), turned to 180 degrees
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Other:
- board outline added: 60 x 75 mm
